File: toolbox/untitled.kicad_sch (KiCad schematic)
At the start: 10 parts

Commit message: added logic shifting
Parts:
- gave numbers to parts that had none: 10
Other:
- moved on the sheet: D2, Q1, Q2, R2, R3, R4, R5, SW1

Commit message: added p-mosfet prcotection circuit
Other:
- note removed: "ON INDICATOR"
- note removed: "ON-OFF INDICATOR"
Changed lines of the file:
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@@
-    (stroke (width 0) (type default) (color 0 0 0 0))
-  )
-  (polyline (pts (xy 35.56 46.99) (xy 121.92 46.99))
     (stroke (width 0) (type default) (color 0 0 0 0))
   )
@@
     (stroke (width 0) (type default) (color 0 0 0 0))
   )
-  (polyline (pts (xy 142.24 46.99) (xy 247.65 46.99))
-    (stroke (width 0) (type default) (color 0 0 0 0))
-  )
   (wire (pts (xy 72.39 88.9) (xy 72.39 93.98))
     (stroke (width 0) (type default) (color 0 0 0 0))
   )
   (wire (pts (xy 234.95 99.06) (xy 234.95 109.22))
-    (stroke (width 0) (type default) (color 0 0 0 0))
-  )
-  (polyline (pts (xy 247.65 151.13) (xy 142.24 151.13))
     (stroke (width 0) (type default) (color 0 0 0 0))
   )
@@
     (stroke (width 0) (type default) (color 0 0 0 0))
   )
-  (polyline (pts (xy 121.92 46.99) (xy 121.92 151.13))
-    (stroke (width 0) (type default) (color 0 0 0 0))
-  )
   (wire (pts (xy 151.13 72.39) (xy 151.13 91.44))
     (stroke (width 0) (type default) (color 0 0 0 0))
   )
   (wire (pts (xy 72.39 116.84) (xy 72.39 120.65))
-    (stroke (width 0) (type default) (color 0 0 0 0))
-  )
-  (polyline (pts (xy 34.29 151.13) (xy 34.29 46.99))
     (stroke (width 0) (type default) (color 0 0 0 0))
   )
@@
     (stroke (width 0) (type default) (color 0 0 0 0))
   )
-  (polyline (pts (xy 247.65 46.99) (xy 247.65 151.13))
-    (stroke (width 0) (type default) (color 0 0 0 0))
-  )
   (wire (pts (xy 217.17 110.49) (xy 217.17 106.68))
     (stroke (width 0) (type default) (color 0 0 0 0))
   )
   (wire (pts (xy 151.13 91.44) (xy 151.13 110.49))
-    (stroke (width 0) (type default) (color 0 0 0 0))
-  )
-  (polyline (pts (xy 142.24 46.99) (xy 142.24 151.13))
     (stroke (width 0) (type default) (color 0 0 0 0))
   )
@@
     (stroke (width 0) (type default) (color 0 0 0 0))
   )
-  (polyline (pts (xy 121.92 151.13) (xy 34.29 151.13))
-    (stroke (width 0) (type default) (color 0 0 0 0))
-  )
   (wire (pts (xy 201.93 147.32) (xy 201.93 134.62))
     (stroke (width 0) (type default) (color 0 0 0 0))
@@
     (stroke (width 0) (type default) (color 0 0 0 0))
   )
-  (text "ON INDICATOR\n\n" (at 48.26 68.58 0)
-    (effects (font (size 5.27 5.27) (thickness 1.054) bold) (justify left bottom))
-  )
-  (text "ON-OFF INDICATOR\n" (at 149.86 60.96 0)
-    (effects (font (size 5.27 5.27) (thickness 1.054) bold) (justify left bottom))
-  )
   (symbol (lib_id "Transistor_BJT:2N3904") (at 201.93 129.54 90) (unit 1)
